File: pcb/strimdick/streamdeck.kicad_pcb (KiCad board)
At the start: 2 copper layers, 118 x 20 mm, 19 parts

Commit message: cleanup
Other:
- board text added: "james_neko's stream deck v1"
- board text removed: "james_neko's strim dick v1"
Changed lines of the file:
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@@
 		(property ki_fp_filters "Resistor_THT:R_Axial_DIN0207_L6.3mm_D2.5mm*")
 		(sheetname "Root")
-		(sheetfile "strimdick.kicad_sch")
+		(sheetfile "streamdeck.kicad_sch")
 		(attr through_hole)
 		(fp_line
@@
 		(property ki_fp_filters "Resistor_THT:R_Axial_DIN0207_L6.3mm_D2.5mm*")
 		(sheetname "Root")
-		(sheetfile "strimdick.kicad_sch")
+		(sheetfile "streamdeck.kicad_sch")
 		(attr through_hole)
 		(fp_line
@@
 		(property ki_fp_filters "Resistor_THT:R_Axial_DIN0207_L6.3mm_D2.5mm*")
 		(sheetname "Root")
-		(sheetfile "strimdick.kicad_sch")
+		(sheetfile "streamdeck.kicad_sch")
 		(attr through_hole)
 		(fp_line
@@
 		(property ki_fp_filters "Resistor_THT:R_Axial_DIN0207_L6.3mm_D2.5mm*")
 		(sheetname "Root")
-		(sheetfile "strimdick.kicad_sch")
+		(sheetfile "streamdeck.kicad_sch")
 		(attr through_hole)
 		(fp_line
@@
 		(property ki_fp_filters "Resistor_THT:R_Axial_DIN0207_L6.3mm_D2.5mm*")
 		(sheetname "Root")
-		(sheetfile "strimdick.kicad_sch")
+		(sheetfile "streamdeck.kicad_sch")
 		(attr through_hole)
 		(fp_line
@@
 		(property ki_fp_filters "Resistor_THT:R_Axial_DIN0207_L6.3mm_D2.5mm*")
 		(sheetname "Root")
-		(sheetfile "strimdick.kicad_sch")
+		(sheetfile "streamdeck.kicad_sch")
 		(attr through_hole)
 		(fp_line
@@
 		(property ki_fp_filters "Arduino_Nano_Socket")
 		(sheetname "Root")
-		(sheetfile "strimdick.kicad_sch")
+		(sheetfile "streamdeck.kicad_sch")
 		(attr through_hole)
 		(fp_line
@@
 		(property ki_fp_filters "LED_D3.0mm_Clear LED_D3.0mm_Horizontal_O1.27mm_Z2.0mm LED_D3.0mm_Horizontal_O3.81mm_Z2.0mm LED_D3.0mm_Horizontal_O6.35mm_Z2.0mm")
 		(sheetname "Root")
-		(sheetfile "strimdick.kicad_sch")
+		(sheetfile "streamdeck.kicad_sch")
 		(attr through_hole exclude_from_pos_files)
 		(fp_line
@@
 		)
 		(sheetname "Root")
-		(sheetfile "strimdick.kicad_sch")
+		(sheetfile "streamdeck.kicad_sch")
 		(attr through_hole exclude_from_pos_files)
 		(fp_line
@@
 		(property ki_fp_filters "LED_D3.0mm_Clear LED_D3.0mm_Horizontal_O1.27mm_Z2.0mm LED_D3.0mm_Horizontal_O3.81mm_Z2.0mm LED_D3.0mm_Horizontal_O6.35mm_Z2.0mm")
 		(sheetname "Root")
-		(sheetfile "strimdick.kicad_sch")
+		(sheetfile "streamdeck.kicad_sch")
 		(attr through_hole exclude_from_pos_files)
 		(fp_line
@@
 		)
 		(sheetname "Root")
-		(sheetfile "strimdick.kicad_sch")
+		(sheetfile "streamdeck.kicad_sch")
 		(attr through_hole exclude_from_pos_files)
 		(fp_line
@@
 		)
 		(sheetname "Root")
-		(sheetfile "strimdick.kicad_sch")
+		(sheetfile "streamdeck.kicad_sch")
 		(attr through_hole exclude_from_pos_files)
 		(fp_line
@@
 		(property ki_fp_filters "LED_D3.0mm_Clear LED_D3.0mm_Horizontal_O1.27mm_Z2.0mm LED_D3.0mm_Horizontal_O3.81mm_Z2.0mm LED_D3.0mm_Horizontal_O6.35mm_Z2.0mm")
 		(sheetname "Root")
-		(sheetfile "strimdick.kicad_sch")
+		(sheetfile "streamdeck.kicad_sch")
 		(attr through_hole exclude_from_pos_files)
 		(fp_line
@@
 		(property ki_fp_filters "LED_D3.0mm_Clear LED_D3.0mm_Horizontal_O1.27mm_Z2.0mm LED_D3.0mm_Horizontal_O3.81mm_Z2.0mm LED_D3.0mm_Horizontal_O6.35mm_Z2.0mm")
 		(sheetname "Root")
-		(sheetfile "strimdick.kicad_sch")
+		(sheetfile "streamdeck.kicad_sch")
 		(attr through_hole exclude_from_pos_files)
 		(fp_line
@@
 		)
 		(sheetname "Root")
-		(sheetfile "strimdick.kicad_sch")
+		(sheetfile "streamdeck.kicad_sch")
 		(attr through_hole exclude_from_pos_files)
 		(fp_line
@@
 		(property ki_fp_filters "LED_D3.0mm_Clear LED_D3.0mm_Horizontal_O1.27mm_Z2.0mm LED_D3.0mm_Horizontal_O3.81mm_Z2.0mm LED_D3.0mm_Horizontal_O6.35mm_Z2.0mm")
 		(sheetname "Root")
-		(sheetfile "strimdick.kicad_sch")
+		(sheetfile "streamdeck.kicad_sch")
 		(attr through_hole exclude_from_pos_files)
 		(fp_line
@@
 		)
 		(sheetname "Root")
-		(sheetfile "strimdick.kicad_sch")
+		(sheetfile "streamdeck.kicad_sch")
 		(attr through_hole exclude_from_pos_files)
 		(fp_line
@@
 		)
 		(sheetname "Root")
-		(sheetfile "strimdick.kicad_sch")
+		(sheetfile "streamdeck.kicad_sch")
 		(attr through_hole exclude_from_pos_files)
 		(fp_line
@@
 		(property ki_fp_filters "LED_D3.0mm_Clear LED_D3.0mm_Horizontal_O1.27mm_Z2.0mm LED_D3.0mm_Horizontal_O3.81mm_Z2.0mm LED_D3.0mm_Horizontal_O6.35mm_Z2.0mm")
 		(sheetname "Root")
-		(sheetfile "strimdick.kicad_sch")
+		(sheetfile "streamdeck.kicad_sch")
 		(attr through_hole exclude_from_pos_files)
 		(fp_line
@@
 		)
 	)
-	(gr_text "james_neko's strim dick v1"
+	(gr_text "james_neko's stream deck v1"
 		(at 70.5 31 0)
 		(layer "F.SilkS")
